Commit message: Add files via upload

File: AutoBot/urdf/AutoBot.urdf (robot description, URDF)
Before this commit: robot AutoBot, 15 links, 14 joints
Links:
- link base_link: mass 455.170796326795 -> 20
- link base_link_to_Left_wheel: mass 26.146 -> 8
- link base_link_to_Right_wheel: mass 26.146 -> 8
- link caster: mass 30.0 -> 1.0
Joints:
- joint base_link_to_left_camera: origin xyz=0.58 0.5 0.5 rpy=0 0.75 1.5708 -> xyz=0.58 0.3 0.5 rpy=0 0.75 1.5708
- joint base_link_to_right_camera: origin xyz=0.58 -0.5 0.5 rpy=0 0.75 -1.5708 -> xyz=0.58 -0.3 0.5 rpy=0 0.75 -1.5708

Commit message: Add files via upload

File: AutoBot/urdf/AutoBot.urdf (robot description, URDF)
Before this commit: robot AutoBot, 15 links, 14 joints
Joints:
- joint base_link_to_left_camera: origin xyz=0.58 0.3 0.5 rpy=0 0.75 1.5708 -> xyz=0.58 0.5 0.5 rpy=0 0.75 1.5708
- joint base_link_to_right_camera: origin xyz=0.58 -0.3 0.5 rpy=0 0.75 -1.5708 -> xyz=0.58 -0.5 0.5 rpy=0 0.75 -1.5708

Commit message: Add files via upload

File: AutoBot/urdf/AutoBot.urdf (robot description, URDF)
Before this commit: robot AutoBot, 15 links, 14 joints
Joints:
- joint base_link_to_lidar: origin xyz=0.58 0 0.6 rpy=0 6.4 0 -> xyz=0.6 0 0 rpy=0 0 0

Commit message: Add files via upload

File: AutoBot/urdf/AutoBot.urdf (robot description, URDF)
Before this commit: robot AutoBot, 15 links, 14 joints
Links:
- added link optical_depth_cam
- added link optical_lidar
Joints:
- added joint optical_depth_cam_joint: type fixed, parent kinect_cam, child optical_depth_cam, origin xyz=0 0 0 rpy=-1.5708 0 -1.5708
- added joint optical_lidar_joint: type fixed, parent lidar, child optical_lidar, origin xyz=0 0 0 rpy=0 0 0
- joint base_link_to_kinect_cam: origin xyz=0.55 0 0.4 rpy=0 0 0 -> xyz=0.55 0 0.8 rpy=0 0.2617 0
